File: Control.kicad_sch (KiCad schematic)
At the start: 8 parts, among them U3 LFE5U-12F-BG256

Commit message: idk
Changed lines of the file:
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@@
     (effects (font (size 1.27 1.27)) (justify left bottom))
   )
-  (hierarchical_label "R~{RAS}" (shape output) (at 388.62 137.16 180) (fields_autoplaced)
-    (effects (font (size 1.27 1.27)) (justify right))
+  (hierarchical_label "R~{RAS}" (shape output) (at 381 132.08 0) (fields_autoplaced)
+    (effects (font (size 1.27 1.27)) (justify left))
+  )
+  (hierarchical_label "XTX1-" (shape output) (at 381 167.64 0) (fields_autoplaced)
+    (effects (font (size 1.27 1.27)) (justify left))
   )
   (hierarchical_label "CSIZ[1..0]" (shape input) (at 372.11 63.5 180) (fields_autoplaced)
     (effects (font (size 1.27 1.27)) (justify right))
   )
-  (hierarchical_label "RDQM[3..0]" (shape output) (at 388.62 152.4 180) (fields_autoplaced)
-    (effects (font (size 1.27 1.27)) (justify right))
+  (hierarchical_label "RDQM[3..0]" (shape output) (at 381 147.32 0) (fields_autoplaced)
+    (effects (font (size 1.27 1.27)) (justify left))
   )
   (hierarchical_label "IOAoutLE" (shape output) (at 314.96 17.78 180) (fields_autoplaced)
@@
   (hierarchical_label "IOSIZ[1..0]" (shape output) (at 314.96 25.4 180) (fields_autoplaced)
     (effects (font (size 1.27 1.27)) (justify right))
+  )
+  (hierarchical_label "XTX1+" (shape output) (at 381 165.1 0) (fields_autoplaced)
+    (effects (font (size 1.27 1.27)) (justify left))
   )
   (hierarchical_label "CA[31..0]" (shape input) (at 328.93 55.88 0) (fields_autoplaced)
@@
     (effects (font (size 1.27 1.27)) (justify left))
   )
+  (hierarchical_label "XCLK-" (shape output) (at 381 157.48 0) (fields_autoplaced)
+    (effects (font (size 1.27 1.27)) (justify left))
+  )
   (hierarchical_label "C~{RMC}" (shape input) (at 388.62 59.69 180) (fields_autoplaced)
     (effects (font (size 1.27 1.27)) (justify right))
   )
-  (hierarchical_label "R~{CS}[2..0]" (shape output) (at 388.62 129.54 180) (fields_autoplaced)
-    (effects (font (size 1.27 1.27)) (justify right))
+  (hierarchical_label "R~{CS}[2..0]" (shape output) (at 381 127 0) (fields_autoplaced)
+    (effects (font (size 1.27 1.27)) (justify left))
   )
   (hierarchical_label "IO~{BERR}" (shape input) (at 346.71 19.05 0) (fields_autoplaced)
+    (effects (font (size 1.27 1.27)) (justify left))
+  )
+  (hierarchical_label "XTX0-" (shape output) (at 381 162.56 0) (fields_autoplaced)
     (effects (font (size 1.27 1.27)) (justify left))
   )
@@
     (effects (font (size 1.27 1.27)) (justify left))
   )
+  (hierarchical_label "XRX-" (shape input) (at 381 172.72 0) (fields_autoplaced)
+    (effects (font (size 1.27 1.27)) (justify left))
+  )
   (hierarchical_label "RESET~{OE}" (shape output) (at 346.71 13.97 0) (fields_autoplaced)
     (effects (font (size 1.27 1.27)) (justify left))
@@
   )
   (hierarchical_label "CD[31..0]" (shape bidirectional) (at 408.94 43.18 0) (fields_autoplaced)
+    (effects (font (size 1.27 1.27)) (justify left))
+  )
+  (hierarchical_label "X~{OE}" (shape input) (at 381 175.26 0) (fields_autoplaced)
     (effects (font (size 1.27 1.27)) (justify left))
   )
@@
     (effects (font (size 1.27 1.27)) (justify right))
   )
-  (hierarchical_label "RA[12..0]" (shape output) (at 388.62 149.86 180) (fields_autoplaced)
-    (effects (font (size 1.27 1.27)) (justify right))
+  (hierarchical_label "RA[12..0]" (shape output) (at 381 144.78 0) (fields_autoplaced)
+    (effects (font (size 1.27 1.27)) (justify left))
+  )
+  (hierarchical_label "XTX0+" (shape output) (at 381 160.02 0) (fields_autoplaced)
+    (effects (font (size 1.27 1.27)) (justify left))
   )
   (hierarchical_label "~{RESET}" (shape input) (at 346.71 16.51 0) (fields_autoplaced)
@@
     (effects (font (size 1.27 1.27)) (justify right))
   )
-  (hierarchical_label "RCKE" (shape output) (at 388.62 144.78 180) (fields_autoplaced)
-    (effects (font (size 1.27 1.27)) (justify right))
+  (hierarchical_label "RCKE" (shape output) (at 381 139.7 0) (fields_autoplaced)
+    (effects (font (size 1.27 1.27)) (justify left))
   )
-  (hierarchical_label "RCLK[5..0]" (shape output) (at 388.62 154.94 180) (fields_autoplaced)
-    (effects (font (size 1.27 1.27)) (justify right))
+  (hierarchical_label "RCLK[5..0]" (shape output) (at 381 149.86 0) (fields_autoplaced)
+    (effects (font (size 1.27 1.27)) (justify left))
   )
-  (hierarchical_label "CASTERM~{EN}" (shape output) (at 388.62 109.22 180) (fields_autoplaced)
-    (effects (font (size 1.27 1.27)) (justify right))
+  (hierarchical_label "CASTERM~{EN}" (shape output) (at 381 109.22 0) (fields_autoplaced)
+    (effects (font (size 1.27 1.27)) (justify left))
   )
-  (hierarchical_label "CCLK" (shape output) (at 387.35 95.25 180) (fields_autoplaced)
-    (effects (font (size 1.27 1.27)) (justify right))
+  (hierarchical_label "CCLK" (shape output) (at 381 101.6 0) (fields_autoplaced)
+    (effects (font (size 1.27 1.27)) (justify left))
   )
-  (hierarchical_label "FCLK" (shape output) (at 387.35 97.79 180) (fields_autoplaced)
-    (effects (font (size 1.27 1.27)) (justify right))
-  )
-  (hierarchical_label "VD[6..0]" (shape output) (at 388.62 162.56 180) (fields_autoplaced)
-    (effects (font (size 1.27 1.27)) (justify right))
+  (hierarchical_label "FCLK" (shape output) (at 381 104.14 0) (fields_autoplaced)
+    (effects (font (size 1.27 1.27)) (justify left))
   )
   (hierarchical_label "IO~{DSACK}1" (shape input) (at 346.71 26.67 0) (fields_autoplaced)
@@
     (effects (font (size 1.27 1.27)) (justify right))
   )
-  (hierarchical_label "R~{CAS}" (shape output) (at 388.62 139.7 180) (fields_autoplaced)
-    (effects (font (size 1.27 1.27)) (justify right))
+  (hierarchical_label "R~{CAS}" (shape output) (at 381 134.62 0) (fields_autoplaced)
+    (effects (font (size 1.27 1.27)) (justify left))
   )
   (hierarchical_label "IO~{CBREQ}" (shape output) (at 314.96 33.02 0) (fields_autoplaced)
     (effects (font (size 1.27 1.27)) (justify left))
   )
-  (hierarchical_label "BA[1..0]" (shape output) (at 388.62 147.32 180) (fields_autoplaced)
-    (effects (font (size 1.27 1.27)) (justify right))
+  (hierarchical_label "BA[1..0]" (shape output) (at 381 142.24 0) (fields_autoplaced)
+    (effects (font (size 1.27 1.27)) (justify left))
   )
-  (hierarchical_label "R~{WE}" (shape output) (at 388.62 142.24 180) (fields_autoplaced)
-    (effects (font (size 1.27 1.27)) (justify right))
+  (hierarchical_label "R~{WE}" (shape output) (at 381 137.16 0) (fields_autoplaced)
+    (effects (font (size 1.27 1.27)) (justify left))
   )
   (hierarchical_label "IOSoutLE" (shape output) (at 314.96 20.32 180) (fields_autoplaced)
     (effects (font (size 1.27 1.27)) (justify right))
   )
-  (hierarchical_label "VCLK" (shape output) (at 388.62 165.1 180) (fields_autoplaced)
-    (effects (font (size 1.27 1.27)) (justify right))
+  (hierarchical_label "C~{BERR}" (shape output) (at 381 121.92 0) (fields_autoplaced)
+    (effects (font (size 1.27 1.27)) (justify left))
   )
-  (hierarchical_label "C~{BERR}" (shape output) (at 387.35 121.92 180) (fields_autoplaced)
-    (effects (font (size 1.27 1.27)) (justify right))
+  (hierarchical_label "XRX+" (shape input) (at 381 170.18 0) (fields_autoplaced)
+    (effects (font (size 1.27 1.27)) (justify left))
   )
-  (hierarchical_label "CS~{STERM}" (shape output) (at 387.35 111.76 180) (fields_autoplaced)
-    (effects (font (size 1.27 1.27)) (justify right))
+  (hierarchical_label "CS~{STERM}" (shape output) (at 381 111.76 0) (fields_autoplaced)
+    (effects (font (size 1.27 1.27)) (justify left))
   )
   (hierarchical_label "IO~{HALT}" (shape input) (at 346.71 21.59 0) (fields_autoplaced)
     (effects (font (size 1.27 1.27)) (justify left))
   )
-  (hierarchical_label "C~{CIIN}" (shape output) (at 387.35 116.84 180) (fields_autoplaced)
-    (effects (font (size 1.27 1.27)) (justify right))
+  (hierarchical_label "C~{CIIN}" (shape output) (at 381 116.84 0) (fields_autoplaced)
+    (effects (font (size 1.27 1.27)) (justify left))
   )
   (hierarchical_label "CD~{OE}" (shape output) (at 406.4 25.4 180) (fields_autoplaced)
     (effects (font (size 1.27 1.27)) (justify right))
   )
-  (hierarchical_label "C~{CBACK}" (shape output) (at 387.35 114.3 180) (fields_autoplaced)
-    (effects (font (size 1.27 1.27)) (justify right))
+  (hierarchical_label "XCLK+" (shape output) (at 381 154.94 0) (fields_autoplaced)
+    (effects (font (size 1.27 1.27)) (justify left))
+  )
+  (hierarchical_label "C~{CBACK}" (shape output) (at 381 114.3 0) (fields_autoplaced)
+    (effects (font (size 1.27 1.27)) (justify left))
   )
   (symbol (lib_id "Device:C_Small") (at 139.7 213.36 0) (unit 1)
