File: MC68k.kicad_sch (KiCad schematic)
At the start: 14 parts, among them U1 MC68030RC, U2 MC68882FN, U22 74LVC138APW, U23 74LVC138APW, U30 741G3208GW, U31 74LVC1G332GW, U32 74LVC1G332GW, U33 741G08GW

Commit message: idk
Parts:
- removed R3, R4: 47, symbol Device:R_Small
- removed U33: 741G08GW, stdpads:SOT-353, symbol GW_Logic:741G08GW
Connections:
- net ~{AS}: now also U32.6 (C)
Changed lines of the file:
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@@
   (junction (at 63.5 187.96) (diameter 0) (color 0 0 0 0)
   )
-  (junction (at 238.76 87.63) (diameter 0) (color 0 0 0 0)
-  )
   (junction (at 66.04 167.64) (diameter 0) (color 0 0 0 0)
   )
@@
   )
   (junction (at 142.24 26.67) (diameter 0) (color 0 0 0 0)
-  )
-  (junction (at 210.82 93.98) (diameter 0) (color 0 0 0 0)
   )
   (junction (at 147.32 177.8) (diameter 0) (color 0 0 0 0)
@@
     (stroke (width 0) (type default))
   )
-  (wire (pts (xy 238.76 99.06) (xy 237.49 99.06))
-    (stroke (width 0) (type default))
-  )
   (bus (pts (xy 99.06 82.55) (xy 99.06 85.09))
     (stroke (width 0) (type default))
@@
     (stroke (width 0) (type default))
   )
-  (wire (pts (xy 204.47 93.98) (xy 210.82 93.98))
-    (stroke (width 0) (type default))
-  )
   (wire (pts (xy 132.08 177.8) (xy 134.62 177.8))
     (stroke (width 0) (type default))
@@
     (stroke (width 0) (type default))
   )
-  (wire (pts (xy 223.52 87.63) (xy 238.76 87.63))
-    (stroke (width 0) (type default))
-  )
   (wire (pts (xy 77.47 133.35) (xy 82.55 133.35))
     (stroke (width 0) (type default))
@@
     (stroke (width 0) (type default))
   )
-  (wire (pts (xy 204.47 92.71) (xy 204.47 93.98))
-    (stroke (width 0) (type default))
-  )
   (bus (pts (xy 85.09 148.59) (xy 85.09 151.13))
     (stroke (width 0) (type default))
@@
     (stroke (width 0) (type default))
   )
-  (wire (pts (xy 238.76 58.42) (xy 238.76 87.63))
-    (stroke (width 0) (type default))
-  )
   (wire (pts (xy 104.14 62.23) (xy 106.68 62.23))
     (stroke (width 0) (type default))
@@
     (stroke (width 0) (type default))
   )
-  (wire (pts (xy 238.76 87.63) (xy 238.76 99.06))
-    (stroke (width 0) (type default))
-  )
   (wire (pts (xy 132.08 26.67) (xy 134.62 26.67))
     (stroke (width 0) (type default))
@@
     (stroke (width 0) (type default))
   )
-  (wire (pts (xy 205.74 92.71) (xy 204.47 92.71))
+  (wire (pts (xy 242.57 60.96) (xy 241.3 60.96))
     (stroke (width 0) (type default))
   )
@@
     (stroke (width 0) (type default))
   )
-  (wire (pts (xy 232.41 99.06) (xy 231.14 99.06))
-    (stroke (width 0) (type default))
-  )
   (bus (pts (xy 99.06 80.01) (xy 99.06 82.55))
     (stroke (width 0) (type default))
@@
     (stroke (width 0) (type default))
   )
+  (wire (pts (xy 241.3 58.42) (xy 246.38 58.42))
+    (stroke (width 0) (type default))
+  )
   (wire (pts (xy 106.68 100.33) (xy 101.6 100.33))
     (stroke (width 0) (type default))
@@
     (stroke (width 0) (type default))
   )
-  (wire (pts (xy 238.76 58.42) (xy 246.38 58.42))
-    (stroke (width 0) (type default))
-  )
   (bus (pts (xy 182.88 144.78) (xy 182.88 147.32))
     (stroke (width 0) (type default))
@@
     (stroke (width 0) (type default))
   )
-  (wire (pts (xy 210.82 93.98) (xy 210.82 87.63))
-    (stroke (width 0) (type default))
-  )
   (bus (pts (xy 85.09 151.13) (xy 85.09 153.67))
     (stroke (width 0) (type default))
@@
     (stroke (width 0) (type default))
   )
-  (wire (pts (xy 210.82 87.63) (xy 218.44 87.63))
-    (stroke (width 0) (type default))
-  )
   (wire (pts (xy 77.47 138.43) (xy 82.55 138.43))
     (stroke (width 0) (type default))
@@
   )
   (wire (pts (xy 106.68 130.81) (xy 101.6 130.81))
+    (stroke (width 0) (type default))
+  )
+  (wire (pts (xy 241.3 60.96) (xy 241.3 58.42))
     (stroke (width 0) (type default))
   )
@@
     (effects (font (size 1.27 1.27)) (justify right))
   )
-  (hierarchical_label "CPUCLK" (shape input) (at 210.82 96.52 180) (fields_autoplaced)
-    (effects (font (size 1.27 1.27)) (justify right))
-  )
   (hierarchical_label "FC[2..0]" (shape output) (at 97.79 39.37 180) (fields_autoplaced)
     (effects (font (size 1.27 1.27)) (justify right))
@@
     (effects (font (size 1.27 1.27)) (justify left))
   )
-  (hierarchical_label "~{AS}" (shape output) (at 205.74 92.71 0) (fields_autoplaced)
+  (hierarchical_label "~{AS}" (shape output) (at 242.57 60.96 0) (fields_autoplaced)
     (effects (font (size 1.27 1.27)) (justify left))
   )
@@
         (path "/70f3c4d7-2986-471b-b5fa-d888368dbdd8/00000000-0000-0000-0000-00005f72f108"
           (reference "U30") (unit 1)
-        )
-      )
-    )
-  )
-  (symbol (lib_id "power:+3V3") (at 231.14 93.98 0) (unit 1)
-    (in_bom yes) (on_board yes) (dnp no)
-    (property "Reference" "#PWR025" (at 231.14 97.79 0)
-      (effects (font (size 1.27 1.27)) hide)
-    )
-    (property "Value" "+3V3" (at 231.14 90.17 0)
-      (effects (font (size 1.27 1.27)))
-    )
-    (property "Footprint" "" (at 231.14 93.98 0)
-      (effects (font (size 1.27 1.27)) hide)
-    )
-    (property "Datasheet" "" (at 231.14 93.98 0)
-      (effects (font (size 1.27 1.27)) hide)
-    )
-    (pin "1")
-    (instances
-      (project "SE-030"
-        (path "/70f3c4d7-2986-471b-b5fa-d888368dbdd8/00000000-0000-0000-0000-00005f72f108"
-          (reference "#PWR025") (unit 1)
         )
       )
@@
     )
   )
-  (symbol (lib_id "GW_Logic:741G08GW") (at 220.98 96.52 0) (unit 1)
-    (in_bom yes) (on_board yes) (dnp no)
-    (property "Reference" "U33" (at 220.98 96.52 0)
-      (effects (font (size 1.27 1.27)))
-    )
-    (property "Value" "741G08GW" (at 220.98 102.87 0)
-      (effects (font (size 1.27 1.27)))
-    )
-    (property "Footprint" "stdpads:SOT-353" (at 220.98 104.14 0)
-      (effects (font (size 1.27 1.27)) (justify top) hide)
-    )
-    (property "Datasheet" "" (at 220.98 101.6 0)
-      (effects (font (size 1.524 1.524)) hide)
-    )
-    (pin "1")
-    (pin "2")
-    (pin "3")
-    (pin "4")
-    (pin "5")
-    (instances
-      (project "SE-030"
-        (path "/70f3c4d7-2986-471b-b5fa-d888368dbdd8/00000000-0000-0000-0000-00005f72f108"
-          (reference "U33") (unit 1)
-        )
-      )
-    )
-  )
   (symbol (lib_id "power:+3V3") (at 210.82 30.48 0) (unit 1)
     (in_bom yes) (on_board yes) (dnp no) (fields_autoplaced)
@@
         (path "/70f3c4d7-2986-471b-b5fa-d888368dbdd8/00000000-0000-0000-0000-00005f72f108"
           (reference "#PWR015") (unit 1)
-        )
-      )
-    )
-  )
-  (symbol (lib_id "power:GND") (at 210.82 99.06 0) (unit 1)
-    (in_bom yes) (on_board yes) (dnp no)
-    (property "Reference" "#PWR026" (at 210.82 105.41 0)
-      (effects (font (size 1.27 1.27)) hide)
-    )
-    (property "Value" "GND" (at 210.82 102.87 0)
-      (effects (font (size 1.27 1.27)))
-    )
-    (property "Footprint" "" (at 210.82 99.06 0)
-      (effects (font (size 1.27 1.27)) hide)
-    )
-    (property "Datasheet" "" (at 210.82 99.06 0)
-      (effects (font (size 1.27 1.27)) hide)
-    )
-    (pin "1")
-    (instances
-      (project "SE-030"
-        (path "/70f3c4d7-2986-471b-b5fa-d888368dbdd8/00000000-0000-0000-0000-00005f72f108"
-          (reference "#PWR026") (unit 1)
         )
       )
@@
     )
   )
-  (symbol (lib_id "Device:R_Small") (at 234.95 99.06 90) (unit 1)
-    (in_bom yes) (on_board yes) (dnp no)
-    (property "Reference" "R4" (at 234.95 97.79 90)
-      (effects (font (size 1.27 1.27)) (justify top))
-    )
-    (property "Value" "47" (at 234.95 100.33 90)
-      (effects (font (size 1.27 1.27)) (justify bottom))
-    )
-    (property "Footprint" "" (at 234.95 99.06 0)
-      (effects (font (size 1.27 1.27)) hide)
-    )
-    (property "Datasheet" "~" (at 234.95 99.06 0)
-      (effects (font (size 1.27 1.27)) hide)
-    )
-    (pin "1")
-    (pin "2")
-    (instances
-      (project "SE-030"
-        (path "/70f3c4d7-2986-471b-b5fa-d888368dbdd8/00000000-0000-0000-0000-00005f72f108"
-          (reference "R4") (unit 1)
-        )
-      )
-    )
-  )
   (symbol (lib_id "power:+3V3") (at 210.82 60.96 0) (unit 1)
     (in_bom yes) (on_board yes) (dnp no) (fields_autoplaced)
@@
         )
       )
-    )
-  )
-  (symbol (lib_id "Device:R_Small") (at 220.98 87.63 90) (unit 1)
-    (in_bom yes) (on_board yes) (dnp no)
-    (property "Reference" "R3" (at 220.98 86.36 90)
-      (effects (font (size 1.27 1.27)) (justify top))
-    )
-    (property "Value" "47" (at 220.98 88.9 90)
-      (effects (font (size 1.27 1.27)) (justify bottom))
-    )
-    (property "Footprint" "" (at 220.98 87.63 0)
-      (effects (font (size 1.27 1.27)) hide)
-    )
-    (property "Datasheet" "~" (at 220.98 87.63 0)
-      (effects (font (size 1.27 1.27)) hide)
-    )
-    (pin "1")
-    (pin "2")
-    (instances
-      (project "SE-030"
-        (path "/70f3c4d7-2986-471b-b5fa-d888368dbdd8/00000000-0000-0000-0000-00005f72f108"
-          (reference "R3") (unit 1)
-        )
-      )
