File: SE-030.kicad_pcb (KiCad board)
At the start: 4 copper layers, 82.7 x 136.5 mm, 165 parts, among them U1 MC68030FE, U10 74AHCT573PW, U11 74AHCT573PW, U12 74AHCT573PW, U13 74LVC244APW, U14 74AHC245APW, U15 74AHC245APW, U16 74AHC245APW, U17 74AHC245APW, U18 74LVC244, U19 74LVC244, U2 MC68882FN, U20 74LVC244, U21 74LVC244, U22 74AHCT573PW, U23 74LVC244APW, U24 74LVC244APW, U25 74AHC245APW, U26 74AHC245APW, U27 74AHC245APW, U28 74AHC245APW, U29 74LVC1G125GW, U3 XC6SLX9-FTG256, U4 W9825G6KH-6, U5 W9825G6KH-6, U6 50M, U8 74AHCT573PW, U9 74AHCT573PW

Commit message: idk
Parts:
- removed the REF** at (243.6, 174.0)

Commit message: lots
Parts:
- removed the REF** at (209.7, 38.8)
- removed the REF** at (233.8, 100.0)
- removed the REF** at (202.6, 38.8)
- removed the REF** at (217.8, 38.8)
- removed the REF** at (199.3, 38.8)
- removed the REF** at (214.6, 38.8)
- removed the REF** at (219.8, 40.8)
- removed the REF** at (219.8, 59.3)
- removed the REF** at (219.8, 56.0)
- removed the REF** at (219.8, 44.0)
- removed the REF** at (217.8, 61.3)
- removed the REF** at (197.3, 49.0)
- removed the REF** at (209.7, 61.3)
- removed the REF** at (199.4, 61.3)
- removed the REF** at (207.6, 61.3)
- removed the REF** at (203.3, 61.3)
- removed the REF** at (213.6, 61.3)
- removed the REF** at (197.3, 40.8)
- removed the REF** at (197.3, 59.4)
- removed the REF** at (197.3, 56.0)
- removed the REF** at (251.4, 55.6)
- removed the REF** at (197.3, 51.1)
- removed the REF** at (268.4, 73.9)
- removed the REF** at (226.2, 85.8)
- removed the REF** at (226.2, 65.0)
- removed the REF** at (226.2, 75.7)
- removed the REF** at (226.2, 83.2)
- removed the REF** at (226.2, 79.4)
- removed the REF** at (193.2, 77.0)
- removed the REF** at (193.2, 81.8)
- removed the REF** at (207.6, 38.8)
- removed the REF** at (210.9, 81.8)
- removed the REF** at (210.9, 77.0)
- removed the REF** at (208.5, 65.0)
- removed the REF** at (208.5, 75.7)
- removed the REF** at (208.5, 85.8)
- removed the REF** at (208.5, 79.4)
- removed the REF** at (208.5, 83.2)
- removed the REF** at (257.6, 71.3)
- removed the REF** at (219.8, 51.1)
- removed the REF** at (233.8, 119.0)
- removed the REF** at (219.8, 49.0)
- removed the REF** at (209.8, 161.0)
- removed the REF** at (212.5, 161.0)
- removed the REF** at (204.9, 161.0)
- removed the REF** at (192.2, 156.0)
- removed the REF** at (192.2, 149.3)
- removed the REF** at (192.2, 135.6)
- removed the REF** at (222.9, 155.5)
- removed the REF** at (194.1, 45.0)
- removed the REF** at (222.9, 148.7)
- removed the REF** at (223.0, 135.6)
- removed the REF** at (193.2, 85.6)
- removed the REF** at (257.6, 115.6)
- removed the REF** at (257.6, 106.8)
- removed the REF** at (257.6, 97.9)
- removed the REF** at (257.6, 89.0)
- removed the REF** at (194.1, 43.5)
- removed the REF** at (257.6, 80.2)
- removed the REF** at (257.6, 133.3)
- removed the REF** at (257.6, 124.5)
- removed the REF** at (257.6, 151.0)
- removed the REF** at (257.6, 142.2)
- removed the REF** at (197.3, 44.0)
- removed the U4 at (200.8, 74.9)
- removed the U6 at (229.2, 54.9)
- added C1: 100n, stdpads:C_0402, F.Cu at (234.6, 178.3)
- added C2: 100n, stdpads:C_0402, F.Cu at (47.9, 44.4)
- added C3: 47u, stdpads:C_1210, F.Cu at (43.5, 45.6)
- added C47: 47u, stdpads:C_1210, F.Cu at (43.5, 50.1)
- added C48: 10n, stdpads:C_0402, F.Cu at (47.9, 46.5)
- added C49: 1n, stdpads:C_0402, F.Cu at (47.9, 48.5)
- added C50: 47p, stdpads:C_0402, F.Cu at (47.9, 50.6)
- added C51: 47p, stdpads:C_0402, F.Cu at (244.0, 179.5)
- added C52: 1n, stdpads:C_0402, F.Cu at (245.1, 179.5)
- added C53: 10n, stdpads:C_0402, F.Cu at (234.6, 181.8)
- added C54: 100n, stdpads:C_0402, F.Cu at (236.6, 175.5)
- added C55: 47u, stdpads:C_1210, F.Cu at (43.5, 54.5)
- added C56: 47u, stdpads:C_1210, F.Cu at (43.5, 59.0)
- added C57: 10u, stdpads:C_0805, F.Cu at (230.9, 177.9)
- added C58: 10u, stdpads:C_0805, F.Cu at (233.0, 177.9)
- added C59: 10u, stdpads:C_0805, F.Cu at (296.9, 92.5)
- added C60: 10u, stdpads:C_0805, F.Cu at (296.9, 95.5)
- added C61: 100n, stdpads:C_0402, F.Cu at (300.7, 87.9)
- added D1: B340LB, stdpads:D_SMA, F.Cu at (61.5, 45.7)
- added D2: B340LB, stdpads:D_SMA, F.Cu at (241.1, 174.6)
- added J2: MacLCPDS, stdpads:DIN41612_R_3x32_Male_Vertical_THT, B.Cu at (268.4, 73.9)
- added L1: 4u7, stdpads:TaiyoYuden_NRS6028, F.Cu at (53.5, 47.2)
- added L2: 4u7, stdpads:TaiyoYuden_NRS6028, F.Cu at (248.0, 174.9)
- added R10: 29k4, stdpads:R_0603, F.Cu at (244.5, 181.4)
- added R11: Rl, stdpads:R_0603, F.Cu at (231.6, 181.1)
- added R12: Rl, stdpads:R_0603, F.Cu at (233.2, 181.1)
- added R13: 3k3, stdpads:R_0603, F.Cu at (248.3, 180.7)
- added R14: 8k2, stdpads:R_0603, F.Cu at (246.8, 180.7)
- added R5: 3k3, stdpads:R_0603, F.Cu at (38.6, 44.6)
- added R6: 10k, stdpads:R_0603, F.Cu at (38.6, 47.1)
- added R7: 29k4, stdpads:R_0603, F.Cu at (38.6, 49.5)
- added R8: Rl, stdpads:R_0603, F.Cu at (44.0, 63.2)
- added R9: Rl, stdpads:R_0603, F.Cu at (44.0, 66.0)
- added REF**: C_0402, stdpads:C_0402, F.Cu at (167.1, 70.8)
- added REF**: C_0402, stdpads:C_0402, F.Cu at (248.1, 132.0)
- added REF**: C_1210, stdpads:C_1210, F.Cu at (242.2, 171.1)
- added REF**: C_0402, stdpads:C_0402, F.Cu at (167.4, 139.6)
- added REF**: SOT-23-6, stdpads:SOT-23-6, F.Cu at (239.3, 188.0)
- added REF**: C_0402, stdpads:C_0402, F.Cu at (182.3, 64.8)
- added REF**: C_0402, stdpads:C_0402, F.Cu at (230.2, 126.1)
- added REF**: C_0402, stdpads:C_0402, F.Cu at (167.1, 60.8)
- added REF**: C_0402, stdpads:C_0402, F.Cu at (182.3, 69.5)
- added REF**: C_0402, stdpads:C_0402, F.Cu at (167.4, 145.9)
- added REF**: C_0402, stdpads:C_0402, F.Cu at (167.1, 63.4)
- added REF**: DIP-32_W15.24mm_LongPads, Package_DIP:DIP-32_W15.24mm_LongPads, F.Cu at (175.3, 221.0)
- added REF**: C_0402, stdpads:C_0402, F.Cu at (230.2, 132.0)
- added REF**: C_0402, stdpads:C_0402, F.Cu at (230.2, 137.9)
- added REF**: Lattice_CABGA-256_14x14mm, stdpads:Lattice_CABGA-256_14x14mm, F.Cu at (192.9, 70.9)
- added REF**: C_0402, stdpads:C_0402, F.Cu at (167.1, 67.2)
- added REF**: DIP-32_W15.24mm_LongPads, Package_DIP:DIP-32_W15.24mm_LongPads, F.Cu at (215.9, 221.0)
- added REF**: DSUB-15-HD_Female_Horizontal_P2.29x1.98mm_EdgePinOffset3.03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, Connector_Dsub:DSUB-15-HD_Female_Horizontal_P2.29x1.98mm_EdgePinOffset3.03mm_Housed_MountingHolesOffset4.94mm, F.Cu at (248.3, 34.8)
- added REF**: C_1210, stdpads:C_1210, F.Cu at (242.2, 167.6)
- added REF**: C_0402, stdpads:C_0402, F.Cu at (167.1, 81.5)
- added REF**: C_0402, stdpads:C_0402, F.Cu at (248.1, 137.9)
- added REF**: DIP-32_W15.24mm_LongPads, Package_DIP:DIP-32_W15.24mm_LongPads, F.Cu at (195.6, 221.0)
- added REF**: DIP-32_W15.24mm_LongPads, Package_DIP:DIP-32_W15.24mm_LongPads, F.Cu at (236.2, 221.0)
- added REF**: C_0402, stdpads:C_0402, F.Cu at (248.1, 126.1)
- added REF**: C_0402, stdpads:C_0402, B.Cu at (235.9, 130.8)
- added REF**: C_0402, stdpads:C_0402, B.Cu at (240.3, 128.8)
- added REF**: C_0402, stdpads:C_0402, B.Cu at (257.6, 90.1)
- added REF**: C_0402, stdpads:C_0402, B.Cu at (257.6, 149.8)
- added REF**: C_0402, stdpads:C_0402, B.Cu at (257.6, 135.1)
- added REF**: C_0402, stdpads:C_0402, B.Cu at (242.3, 130.8)
- added REF**: C_0402, stdpads:C_0402, B.Cu at (242.3, 133.2)
- added REF**: C_0402, stdpads:C_0402, B.Cu at (257.6, 105.1)
- added REF**: C_0402, stdpads:C_0402, B.Cu at (241.2, 105.0)
- added REF**: C_0402, stdpads:C_0402, B.Cu at (239.2, 133.7)
- added REF**: C_0402, stdpads:C_0402, B.Cu at (257.6, 142.6)
- added REF**: C_0402, stdpads:C_0402, B.Cu at (250.1, 105.9)
- added REF**: C_0402, stdpads:C_0402, B.Cu at (237.9, 132.0)
- added REF**: C_0402, stdpads:C_0402, B.Cu at (228.2, 105.9)
- added REF**: C_0402, stdpads:C_0402, B.Cu at (257.6, 120.1)
- added REF**: C_0402, stdpads:C_0402, B.Cu at (243.7, 105.9)
- added REF**: C_0402, stdpads:C_0402, B.Cu at (237.9, 128.8)
- added REF**: C_0402, stdpads:C_0402, B.Cu at (239.6, 135.2)
- added REF**: C_0402, stdpads:C_0402, B.Cu at (240.8, 132.0)
- added REF**: C_0402, stdpads:C_0402, B.Cu at (257.6, 75.3)
- added REF**: C_0402, stdpads:C_0402, B.Cu at (237.6, 135.2)
- added REF**: C_0402, stdpads:C_0402, B.Cu at (257.6, 82.6)
- added REF**: C_0402, stdpads:C_0402, B.Cu at (239.2, 130.3)
- added REF**: C_0402, stdpads:C_0402, B.Cu at (257.6, 112.6)
- added REF**: C_0402, stdpads:C_0402, B.Cu at (247.4, 105.9)
- added REF**: C_0402, stdpads:C_0402, B.Cu at (257.6, 97.6)
- added REF**: C_0402, stdpads:C_0402, B.Cu at (235.9, 133.2)
- added REF**: C_0402, stdpads:C_0402, B.Cu at (257.6, 127.6)
- added REF**: C_0402, stdpads:C_0402, B.Cu at (238.7, 105.9)
- added U10: 74AHCT573PW, stdpads:TSSOP-20_4.4x6.5mm_P0.65mm, F.Cu at (255.2, 152.6)
- added U30: 741G3208GW, stdpads:SOT-363, F.Cu at (69.7, 45.2)
- added U31: 74LVC1G332GW, stdpads:SOT-363, F.Cu at (69.7, 48.9)
- added U32: 74LVC1G332GW, stdpads:SOT-363, F.Cu at (69.7, 52.5)
- added U33: 741G08GW, stdpads:SOT-353, F.Cu at (69.7, 56.2)
- added U34: 74AHCT573PW, stdpads:TSSOP-20_4.4x6.5mm_P0.65mm, F.Cu at (255.2, 78.1)
- added U35: TPS54331D, stdpads:SOIC-8_3.9mm, F.Cu at (52.8, 63.1)
- added U36: TPS54331D, stdpads:SOIC-8_3.9mm, F.Cu at (239.1, 179.4)
- added U4: W9825G6KH-6, stdpads:TSOP-II-54_22.2x10.16mm_P0.8mm, F.Cu at (239.2, 113.4)
- added U4: W9825G6KH-6, stdpads:TSOP-II-54_22.2x10.16mm_P0.8mm, F.Cu at (174.7, 71.7)
- added U7: 74LVC244APW, stdpads:TSSOP-20_4.4x6.5mm_P0.65mm, F.Cu at (40.8, 83.8)
- U1: value MC68030FE -> MC68030RC; footprint stdpads:PQFP-132_24x24mm_P0.635mm_MC68030 -> stdpads:PGA-128_MC68030
- U13: renamed from U17; value 74AHC245APW -> 74LVC245APW
- U14: renamed from U10; value 74AHCT573PW -> 74AHC245APW
- U18, U19, U20, U21: value 74LVC244 -> 74LVC244APW
- U22: value 74AHCT573PW -> 74LVC138APW; footprint stdpads:TSSOP-20_4.4x6.5mm_P0.65mm -> stdpads:TSSOP-16_4.4x5mm_P0.65mm
- U23: value 74LVC244APW -> 74LVC138APW; footprint stdpads:TSSOP-20_4.4x6.5mm_P0.65mm -> stdpads:TSSOP-16_4.4x5mm_P0.65mm
- U3: value XC6SLX9-FTG256 -> LFE5U-12F-BG256; footprint Package_BGA:BGA-256_17.0x17.0mm_Layout16x16_P1.0mm_Ball0.5mm_Pad0.4mm_NSMD -> stdpads:Lattice_CABGA-256_14x14mm
- U6: renamed from U13; value 74LVC244APW -> 74AHCT573PW
- moved U23 167.3 mm to (82.0, 47.9), turned to 0 degrees
- moved U22 166.0 mm to (75.2, 47.9), turned to 0 degrees
- moved C39 159.2 mm to (42.5, 70.8)
- moved C12 153.4 mm to (74.0, 53.9)
- moved C13 153.4 mm to (74.0, 56.9)
- moved C43 152.2 mm to (46.3, 70.8)
- moved C44 151.1 mm to (46.3, 73.2)
- moved C14 150.8 mm to (74.0, 60.0)
- moved C15 150.8 mm to (74.0, 63.0)
- moved C35 150.4 mm to (38.6, 70.8)
- moved C36 150.4 mm to (38.6, 73.2)
- moved C40 150.4 mm to (42.5, 73.2)
- moved C45 150.4 mm to (46.3, 75.7)
- moved C37 149.4 mm to (38.6, 75.7)
- moved C41 149.4 mm to (42.5, 75.7)
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- renumbered U14 to U15, U15 to U16, U16 to U17
Connections:
- net /CPUBuf/FSB_~RMC~ renamed /CPUBuf/C~{RMC}
- net /Control/CCLK_SCK renamed /Control/TDI
- net /Control/CPU_D~OE~ renamed /Control/CPU_D~{OE}
- net /Control/FPU~CS~ renamed /Control/FPU~{CS}
- net /Control/IOB_~DSACK~1 renamed /PDSBuf/LRMC
- net /Control/M0 renamed /Control/TMS
- net /Control/RESET~OE~ renamed /Control/RESET~{OE}
- net /PDSBuf/IOB_SIZ1 renamed /PDSBuf/L~{RMC}
- net /PDSBuf/IOB_~AS~ renamed /PDS/~{FAN}
- net /PDSBuf/IOC_A0 renamed /PDSBuf/AD2
- net Net-(U24-Pad5) renamed /CPUBuf/CFC0
- net Net-(U24-Pad7) renamed /CPUBuf/CSIZ0
- net Net-(U24-Pad9) renamed /CPUBuf/CSIZ1
- net Net-(U3-PadM10) renamed /Control/TDO
- net Net-(U3-PadR9) renamed /Control/~{PROG}
- net Net-(U3-PadT10) renamed /Control/TCK
- net Net-(U3-PadT7) renamed /Control/MISO
- net Net-(U3-PadT8) renamed /Control/MOSI
- net Net-(U3-PadT9) renamed /Control/~{INIT}
- U11 pad 1: /PDSBuf/A~OE~ -> /Control/IOA~{OE}
- U11 pad 11: /PDSBuf/ADoutLE -> /PDSBuf/AoutLE
- U11 pad 12: /PDS/A8 -> /PDS/A15
- U11 pad 13: /PDS/A9 -> /PDS/A16
- U11 pad 14: /PDS/A10 -> /PDS/A17
- U11 pad 15: /PDS/A11 -> /PDS/A18
- U11 pad 16: /PDS/A12 -> /PDS/A19
- U11 pad 17: /PDS/A13 -> /PDS/A20
- U11 pad 18: /PDS/A14 -> /PDS/A21
- U11 pad 19: /PDS/A15 -> /PDS/A22
- U11 pad 2: /CPUBuf/FSB_A15 -> /PDSBuf/FSB_A15
- U11 pad 3: /CPUBuf/FSB_A14 -> /PDSBuf/FSB_A14
- U11 pad 4: /CPUBuf/FSB_A13 -> /PDSBuf/FSB_A13
- U11 pad 5: /CPUBuf/FSB_A12 -> /PDSBuf/FSB_A12
- U11 pad 6: /CPUBuf/FSB_A11 -> /PDSBuf/FSB_A11
- U11 pad 7: /CPUBuf/FSB_A10 -> /PDSBuf/FSB_A10
- U11 pad 8: /CPUBuf/FSB_A9 -> /PDSBuf/FSB_A9
- U11 pad 9: /CPUBuf/FSB_A8 -> /PDSBuf/FSB_A8
- U12 pad 1: /PDSBuf/A~OE~ -> /Control/IOA~{OE}
- U12 pad 11: /PDSBuf/ADoutLE -> /PDSBuf/AoutLE
- U12 pad 12: /PDSBuf/IOB_FC0 -> /PDS/A23
- U12 pad 13: /PDSBuf/IOB_FC1 -> /PDS/A24
- U12 pad 14: /PDSBuf/IOB_FC2 -> /PDS/A25
- U12 pad 15: /PDSBuf/IOB_~RMC~ -> /PDS/A26
- U12 pad 16: /PDS/A4 -> /PDS/A27
- U12 pad 17: /PDS/A5 -> /PDS/A31
- U12 pad 18: /PDS/A6 -> /PDS/A1
- U12 pad 19: /PDS/A7 -> /PDS/A0
- U12 pad 2: /CPUBuf/FSB_A7 -> /PDSBuf/AD0
- U12 pad 3: /CPUBuf/FSB_A6 -> /PDSBuf/AD1
- U12 pad 4: /CPUBuf/FSB_A5 -> /PDSBuf/AD31
- U12 pad 5: /CPUBuf/FSB_A4 -> /PDSBuf/AD3
- U12 pad 6: +5V -> /PDSBuf/AD4
- U12 pad 7: /CPUBuf/FSB_FC2 -> /PDSBuf/AD5
- U12 pad 8: /CPUBuf/FSB_FC1 -> /PDSBuf/AD6
- U12 pad 9: /CPUBuf/FSB_FC0 -> /PDSBuf/AD7
- U13 pad 1: /PDSBuf/DDIR -> GND
- U13 pad 11: /PDS/D31 -> GND
- U13 pad 12: /PDS/D30 -> /MC68k/~{RESET}
- U13 pad 13: /PDS/D29 -> GND
- U13 pad 14: /PDS/D28 -> /PDS/C16M
- U13 pad 15: /PDS/D27 -> GND
- U13 pad 16: /PDS/D26 -> /PDS/~{HALT}
- U13 pad 17: /PDS/D25 -> /PDS/~{DSACK}0
- U13 pad 18: /PDS/D24 -> /PDS/~{DSACK}1
- U13 pad 19: /PDSBuf/D~OE~ -> /PDS/~{BERR}
- U13 pad 2: /PDSBuf/IOC_D24 -> /Control/IO~{BERR}
- U13 pad 3: /PDSBuf/IOC_D25 -> /Control/IO~{DSACK}1
- U13 pad 4: /PDSBuf/IOC_D26 -> /Control/IO~{DSACK}0
- U13 pad 5: /PDSBuf/IOC_D27 -> /Control/IO~{HALT}
- U13 pad 6: /PDSBuf/IOC_D28 -> GND
- U13 pad 7: /PDSBuf/IOC_D29 -> /Control/C16M
- U13 pad 8: /PDSBuf/IOC_D30 -> GND
- U13 pad 9: /PDSBuf/IOC_D31 -> /Control/~{RESET}
- U14 pad 1: /PDSBuf/A~OE~ -> /PDSBuf/DDIR
- U14 pad 11: /PDSBuf/ADoutLE -> /PDS/D7
- U14 pad 12: /PDS/A16 -> /PDS/D0
- U14 pad 13: /PDS/A17 -> /PDS/D1
- U14 pad 14: /PDS/A18 -> /PDS/D6
- U14 pad 15: /PDS/A19 -> /PDS/D5
- U14 pad 16: /PDS/A20 -> /PDS/D2
- U14 pad 17: /PDS/A21 -> /PDS/D4
- U14 pad 18: /PDS/A22 -> /PDS/D3
- U14 pad 19: /PDS/A23 -> /Control/IOD~{OE}
- U14 pad 2: /CPUBuf/FSB_A23 -> /PDSBuf/IOC_D3
- U14 pad 20: +5V -> +3V3
- U14 pad 3: /CPUBuf/FSB_A22 -> /PDSBuf/IOC_D4
- U14 pad 4: /CPUBuf/FSB_A21 -> /PDSBuf/IOC_D2
- U14 pad 5: /CPUBuf/FSB_A20 -> /PDSBuf/IOC_D5
- U14 pad 6: /CPUBuf/FSB_A19 -> /PDSBuf/IOC_D6
- U14 pad 7: /CPUBuf/FSB_A18 -> /PDSBuf/IOC_D1
- U14 pad 8: /CPUBuf/FSB_A17 -> /PDSBuf/IOC_D0
- U14 pad 9: /CPUBuf/FSB_A16 -> /PDSBuf/IOC_D7
- U15 pad 11: /PDS/D7 -> /PDS/D8
- U15 pad 12: /PDS/D6 -> /PDS/D9
- U15 pad 13: /PDS/D5 -> /PDS/D10
- U15 pad 14: /PDS/D4 -> /PDS/D11
- U15 pad 15: /PDS/D3 -> /PDS/D12
- U15 pad 16: /PDS/D2 -> /PDS/D13
- U15 pad 17: /PDS/D1 -> /PDS/D14
- U15 pad 18: /PDS/D0 -> /PDS/D15
- U15 pad 19: /PDSBuf/D~OE~ -> /Control/IOD~{OE}
- U15 pad 2: /PDSBuf/IOC_D0 -> /PDSBuf/IOC_D15
- U15 pad 3: /PDSBuf/IOC_D1 -> /PDSBuf/IOC_D14
- U15 pad 4: /PDSBuf/IOC_D2 -> /PDSBuf/IOC_D13
- U15 pad 5: /PDSBuf/IOC_D3 -> /PDSBuf/IOC_D12
- U15 pad 6: /PDSBuf/IOC_D4 -> /PDSBuf/IOC_D11
- U15 pad 7: /PDSBuf/IOC_D5 -> /PDSBuf/IOC_D10
- U15 pad 8: /PDSBuf/IOC_D6 -> /PDSBuf/IOC_D9
- U15 pad 9: /PDSBuf/IOC_D7 -> /PDSBuf/IOC_D8
- U16 pad 11: /PDS/D15 -> /PDS/D16
- U16 pad 12: /PDS/D14 -> /PDS/D17
- U16 pad 13: /PDS/D13 -> /PDS/D18
- U16 pad 14: /PDS/D12 -> /PDS/D19
- U16 pad 15: /PDS/D11 -> /PDS/D20
- U16 pad 16: /PDS/D10 -> /PDS/D21
- U16 pad 17: /PDS/D9 -> /PDS/D22
- U16 pad 18: /PDS/D8 -> /PDS/D23
- U16 pad 19: /PDSBuf/D~OE~ -> /Control/IOD~{OE}
- U16 pad 2: /PDSBuf/IOC_D8 -> /PDSBuf/IOC_D23
- U16 pad 3: /PDSBuf/IOC_D9 -> /PDSBuf/IOC_D22
- U16 pad 4: /PDSBuf/IOC_D10 -> /PDSBuf/IOC_D21
- U16 pad 5: /PDSBuf/IOC_D11 -> /PDSBuf/IOC_D20
- U16 pad 6: /PDSBuf/IOC_D12 -> /PDSBuf/IOC_D19
- U16 pad 7: /PDSBuf/IOC_D13 -> /PDSBuf/IOC_D18
- U16 pad 8: /PDSBuf/IOC_D14 -> /PDSBuf/IOC_D17
- U16 pad 9: /PDSBuf/IOC_D15 -> /PDSBuf/IOC_D16
- U17 pad 11: /PDS/D23 -> /PDS/D24
- U17 pad 12: /PDS/D22 -> /PDS/D25
- U17 pad 13: /PDS/D21 -> /PDS/D26
- U17 pad 14: /PDS/D20 -> /PDS/D27
- U17 pad 15: /PDS/D19 -> /PDS/D28
- U17 pad 16: /PDS/D18 -> /PDS/D29
- U17 pad 17: /PDS/D17 -> /PDS/D30
- U17 pad 18: /PDS/D16 -> /PDS/D31
- U17 pad 19: /PDSBuf/D~OE~ -> /Control/IOD~{OE}
- U17 pad 2: /PDSBuf/IOC_D16 -> /PDSBuf/IOC_D31
- U17 pad 3: /PDSBuf/IOC_D17 -> /PDSBuf/IOC_D30
- U17 pad 4: /PDSBuf/IOC_D18 -> /PDSBuf/IOC_D29
- U17 pad 5: /PDSBuf/IOC_D19 -> /PDSBuf/IOC_D28
- U17 pad 6: /PDSBuf/IOC_D20 -> /PDSBuf/IOC_D27
- U17 pad 7: /PDSBuf/IOC_D21 -> /PDSBuf/IOC_D26
- U17 pad 8: /PDSBuf/IOC_D22 -> /PDSBuf/IOC_D25
- U17 pad 9: /PDSBuf/IOC_D23 -> /PDSBuf/IOC_D24
- U18 pad 1: /CPUBuf/A~OE~ -> GND
- U18 pad 11: /MC68k/A7 -> /CPUBuf/CPU_A7
- U18 pad 13: /MC68k/A6 -> /CPUBuf/CPU_A6
- U18 pad 15: /MC68k/A5 -> /CPUBuf/CPU_A5
- U18 pad 17: /MC68k/A4 -> /CPUBuf/CPU_A4
- U18 pad 19: /CPUBuf/A~OE~ -> GND
- U18 pad 2: /MC68k/A0 -> /CPUBuf/CPU_A0
- U18 pad 4: /MC68k/A1 -> /CPUBuf/CPU_A1
- U18 pad 6: /MC68k/A2 -> /CPUBuf/CPU_A2
- U18 pad 8: /MC68k/A3 -> /CPUBuf/CPU_A3
- U19 pad 1: /CPUBuf/A~OE~ -> GND
- U19 pad 11: /MC68k/A15 -> /CPUBuf/CPU_A15
- U19 pad 13: /MC68k/A14 -> /CPUBuf/CPU_A14
- U19 pad 15: /MC68k/A13 -> /CPUBuf/CPU_A13
- U19 pad 17: /MC68k/A12 -> /CPUBuf/CPU_A12
- U19 pad 19: /CPUBuf/A~OE~ -> GND
- U19 pad 2: /MC68k/A8 -> /CPUBuf/CPU_A8
- U19 pad 4: /MC68k/A9 -> /CPUBuf/CPU_A9
- U19 pad 6: /MC68k/A10 -> /CPUBuf/CPU_A10
- U19 pad 8: /MC68k/A11 -> /CPUBuf/CPU_A11
- U2 pad 13: /PDSBuf/IOB_~RESET~ -> /PDSBuf/IOB_~{RESET}
- U2 pad 20: /CPUBuf/CPU_~DS~ -> /CPUBuf/CPU_~{DS}
- U2 pad 21: /CPUBuf/CPU_~AS~ -> /CPUBuf/CPU_~{AS}
- U2 pad 28: /CPUBuf/CPU_R~W~ -> /CPUBuf/CPU_R~{W}
- U2 pad 31: /CPUBuf/CPU_~DSACK~0 -> /CPUBuf/CPU_~{DSACK}0
- U2 pad 32: /CPUBuf/CPU_~DSACK~1 -> /CPUBuf/CPU_~{DSACK}1
- U20 pad 1: /CPUBuf/A~OE~ -> GND
- U20 pad 11: /MC68k/A23 -> /CPUBuf/CPU_A23
- U20 pad 13: /MC68k/A22 -> /CPUBuf/CPU_A22
- U20 pad 15: /MC68k/A21 -> /CPUBuf/CPU_A21
- U20 pad 17: /MC68k/A20 -> /CPUBuf/CPU_A20
- U20 pad 19: /CPUBuf/A~OE~ -> GND
- U20 pad 2: /MC68k/A16 -> /CPUBuf/CPU_A16
- U20 pad 4: /MC68k/A17 -> /CPUBuf/CPU_A17
- U20 pad 6: /MC68k/A18 -> /CPUBuf/CPU_A18
- U20 pad 8: /MC68k/A19 -> /CPUBuf/CPU_A19
- U21 pad 1: /CPUBuf/A~OE~ -> GND
- U21 pad 11: /MC68k/A31 -> /CPUBuf/CPU_A31
- U21 pad 13: /MC68k/A30 -> /CPUBuf/CPU_A30
- U21 pad 15: /MC68k/A29 -> /CPUBuf/CPU_A29
- U21 pad 17: /MC68k/A28 -> /CPUBuf/CPU_A28
- U21 pad 19: /CPUBuf/A~OE~ -> GND
- U21 pad 2: /MC68k/A24 -> /CPUBuf/CPU_A24
- U21 pad 4: /MC68k/A25 -> /CPUBuf/CPU_A25
- U21 pad 6: /MC68k/A26 -> /CPUBuf/CPU_A26
- U21 pad 8: /MC68k/A27 -> /CPUBuf/CPU_A27
- U22 pad 1: /CPUBuf/DSACK~OE~ -> /CPUBuf/FC0
- U22 pad 10: GND -> unconnected-(U22-~{Q5}-Pad10)
- U22 pad 11: +3V3 -> unconnected-(U22-~{Q4}-Pad11)
- U22 pad 12: Net-(U22-Pad12) -> unconnected-(U22-~{Q3}-Pad12)
- U22 pad 13: Net-(U22-Pad13) -> unconnected-(U22-~{Q2}-Pad13)
- U22 pad 14: Net-(U22-Pad14) -> unconnected-(U22-~{Q1}-Pad14)
- U22 pad 15: Net-(U22-Pad15) -> unconnected-(U22-~{Q0}-Pad15)
- U22 pad 16: Net-(U22-Pad16) -> +3V3
- U22 pad 2: /Control/CPU_~DSACK~1 -> /CPUBuf/FC1
- U22 pad 3: /Control/CPU_~DSACK~0 -> /CPUBuf/FC2
- U22 pad 4: Net-(U22-Pad4) -> GND
- U22 pad 5: Net-(U22-Pad5) -> /CPUBuf/A19
- U22 pad 6: Net-(U22-Pad6) -> /CPUBuf/A17
- U22 pad 8: Net-(U22-Pad8) -> GND
- U22 pad 9: Net-(U22-Pad9) -> unconnected-(U22-~{Q6}-Pad9)
- U23 pad 1: GND -> /CPUBuf/A16
- U23 pad 10: GND -> unconnected-(U23-~{Q5}-Pad10)
- U23 pad 11: GND -> unconnected-(U23-~{Q4}-Pad11)
- U23 pad 12: /CPUBuf/FSB_~AS~ -> unconnected-(U23-~{Q3}-Pad12)
- U23 pad 13: /CPUBuf/CPU_SIZ1 -> unconnected-(U23-~{Q2}-Pad13)
- U23 pad 14: /CPUBuf/FSB_~CBREQ~ -> unconnected-(U23-~{Q1}-Pad14)
- U23 pad 15: /CPUBuf/CPU_SIZ0 -> Net-(U23-~{Q0})
- U23 pad 16: /CPUBuf/FSB_~DS~ -> +3V3
- U23 pad 2: /CPUBuf/CPU_~AS~ -> /CPUBuf/A15
- U23 pad 3: /CPUBuf/FSB_~CIOUT~ -> /CPUBuf/A14
- U23 pad 4: /CPUBuf/CPU_~CBREQ~ -> GND
- U23 pad 5: /CPUBuf/FSB_SIZ0 -> /CPUBuf/A18
- U23 pad 6: /CPUBuf/CPU_~DS~ -> /CPUBuf/A13
- U23 pad 7: /CPUBuf/FSB_SIZ1 -> unconnected-(U23-~{Q7}-Pad7)
- U23 pad 8: /CPUBuf/CPU_~ECS~ -> GND
- U23 pad 9: Net-(U23-Pad9) -> unconnected-(U23-~{Q6}-Pad9)
- U24 pad 1: /CPUBuf/A~OE~ -> GND
- U24 pad 11: GND -> /CPUBuf/SIZ1
- U24 pad 13: GND -> /CPUBuf/SIZ0
- U24 pad 14: /CPUBuf/FSB_R~W~ -> /CPUBuf/CR~{W}
- U24 pad 15: GND -> /CPUBuf/FC0
- U24 pad 16: /CPUBuf/FSB_FC2 -> /CPUBuf/DDIR
- U24 pad 17: /CPUBuf/CPU_FC0 -> /CPUBuf/FC1
- U24 pad 18: /CPUBuf/FSB_FC1 -> /CPUBuf/CFC2
- U24 pad 19: /CPUBuf/A~OE~ -> GND
- U24 pad 2: /CPUBuf/CPU_~RMC~ -> /CPUBuf/~{RMC}
- U24 pad 3: /CPUBuf/FSB_FC0 -> /CPUBuf/CFC1
- U24 pad 4: /CPUBuf/CPU_R~W~ -> /CPUBuf/R~{W}
- U24 pad 6: /CPUBuf/CPU_FC2 -> /CPUBuf/R~{W}
- U24 pad 8: /CPUBuf/CPU_FC1 -> /CPUBuf/FC2
- U3 pad A10: Net-(U3-PadA10) -> unconnected-(U3B-PT42B-PadA10)
- U3 pad A11: Net-(U3-PadA11) -> unconnected-(U3B-PT53A-PadA11)
- U3 pad A12: Net-(U3-PadA12) -> unconnected-(U3B-PT53B-PadA12)
- U3 pad A13: Net-(U3-PadA13) -> unconnected-(U3B-PT65A-PadA13)
- U3 pad A14: Net-(U3-PadA14) -> unconnected-(U3B-PT65B-PadA14)
- U3 pad A15: Net-(U3-PadA15) -> unconnected-(U3B-PT67B-PadA15)
- U3 pad A2: Net-(U3-PadA2) -> unconnected-(U3A-PT4A-PadA2)
- U3 pad A3: Net-(U3-PadA3) -> unconnected-(U3A-PT6A-PadA3)
- U3 pad A4: Net-(U3-PadA4) -> unconnected-(U3A-PT6B-PadA4)
- U3 pad A5: Net-(U3-PadA5) -> unconnected-(U3A-PT18A-PadA5)
- U3 pad A6: Net-(U3-PadA6) -> unconnected-(U3A-PT18B-PadA6)
- U3 pad A7: Net-(U3-PadA7) -> unconnected-(U3A-PCK00/PT29A-PadA7)
- U3 pad A8: Net-(U3-PadA8) -> unconnected-(U3A-~{PCK}00/PT29B-PadA8)
- U3 pad A9: Net-(U3-PadA9) -> unconnected-(U3B-PT42A-PadA9)
- U3 pad B1: Net-(U3-PadB1) -> unconnected-(U3F-PL2A-PadB1)
- U3 pad B10: Net-(U3-PadB10) -> unconnected-(U3B-PT44A-PadB10)
- U3 pad B11: GND -> unconnected-(U3B-PT49A-PadB11)
- U3 pad B12: Net-(U3-PadB12) -> unconnected-(U3B-PT56A-PadB12)
- U3 pad B13: +3V3 -> unconnected-(U3B-PT60A-PadB13)
- U3 pad B14: Net-(U3-PadB14) -> unconnected-(U3B-PT67A-PadB14)
- U3 pad B15: Net-(U3-PadB15) -> unconnected-(U3C-S0_IN/PR2B-PadB15)
- U3 pad B16: Net-(U3-PadB16) -> unconnected-(U3C-PR2A-PadB16)
- U3 pad B2: Net-(U3-PadB2) -> unconnected-(U3F-PL2B-PadB2)
- U3 pad B3: Net-(U3-PadB3) -> unconnected-(U3A-PT4B-PadB3)
- U3 pad B4: +3V3 -> unconnected-(U3A-PT11B-PadB4)
- U3 pad B5: Net-(U3-PadB5) -> unconnected-(U3A-PT15B-PadB5)
- U3 pad B6: Net-(U3-PadB6) -> unconnected-(U3A-PT22B-PadB6)
- U3 pad B7: GND -> unconnected-(U3A-~{PCK}01/PT27B-PadB7)
- U3 pad B8: Net-(U3-PadB8) -> unconnected-(U3B-~{PCK}10/PT35B-PadB8)
- U3 pad B9: +3V3 -> unconnected-(U3B-GR10/PT38A-PadB9)
- U3 pad C1: Net-(U3-PadC1) -> unconnected-(U3F-PL5A-PadC1)
- U3 pad C10: Net-(U3-PadC10) -> unconnected-(U3B-PT44B-PadC10)
- U3 pad C11: Net-(U3-PadC11) -> unconnected-(U3B-PT49B-PadC11)
- U3 pad C12: Net-(U3-PadC12) -> unconnected-(U3B-PT56B-PadC12)
- U3 pad C13: Net-(U3-PadC13) -> unconnected-(U3B-PT60B-PadC13)
- U3 pad C14: Net-(U3-PadC14) -> unconnected-(U3C-PR2C-PadC14)
- U3 pad C15: Net-(U3-PadC15) -> unconnected-(U3C-PR5B-PadC15)
- U3 pad C16: Net-(U3-PadC16) -> unconnected-(U3C-PR5A-PadC16)
- U3 pad C2: Net-(U3-PadC2) -> unconnected-(U3F-PL5B-PadC2)
- U3 pad C3: Net-(U3-PadC3) -> unconnected-(U3F-PL2C-PadC3)
- U3 pad C4: /Control/HSWAPEN -> unconnected-(U3A-PT11A-PadC4)
- U3 pad C5: Net-(U3-PadC5) -> unconnected-(U3A-PT15A-PadC5)
- U3 pad C6: Net-(U3-PadC6) -> unconnected-(U3A-PT22A-PadC6)
- U3 pad C7: Net-(U3-PadC7) -> unconnected-(U3A-PCK01/PT27A-PadC7)
- U3 pad C8: Net-(U3-PadC8) -> unconnected-(U3B-PCK10/PT35A-PadC8)
- U3 pad C9: Net-(U3-PadC9) -> unconnected-(U3B-GR11/PT38B-PadC9)
- U3 pad D1: Net-(U3-PadD1) -> unconnected-(U3F-PL8A-PadD1)
- U3 pad D10: +3V3 -> unconnected-(U3B-PT47A-PadD10)
- U3 pad D11: Net-(U3-PadD11) -> unconnected-(U3B-PT51A-PadD11)
- U3 pad D12: Net-(U3-PadD12) -> unconnected-(U3B-PT58A-PadD12)
- U3 pad D13: GND -> unconnected-(U3B-PT62A-PadD13)
- U3 pad D14: Net-(U3-PadD14) -> unconnected-(U3C-PR2D-PadD14)
- U3 pad D15: +3V3 -> GND
- U3 pad D16: Net-(U3-PadD16) -> unconnected-(U3C-PR8A-PadD16)
- U3 pad D2: +3V3 -> GND
- U3 pad D3: Net-(U3-PadD3) -> unconnected-(U3F-PL2D-PadD3)
- U3 pad D4: GND -> unconnected-(U3A-PT9B-PadD4)
- U3 pad D5: Net-(U3-PadD5) -> unconnected-(U3A-PT13B-PadD5)
- U3 pad D6: Net-(U3-PadD6) -> unconnected-(U3A-PT20B-PadD6)
- U3 pad D7: +3V3 -> unconnected-(U3A-GR01/PT24B-PadD7)
- U3 pad D8: Net-(U3-PadD8) -> unconnected-(U3B-~{PCK}11/PT33B-PadD8)
- U3 pad D9: Net-(U3-PadD9) -> unconnected-(U3B-PT40A-PadD9)
- U3 pad E1: Net-(U3-PadE1) -> unconnected-(U3F-PL11D-PadE1)
- U3 pad E10: Net-(U3-PadE10) -> unconnected-(U3B-PT47B-PadE10)
- U3 pad E11: Net-(U3-PadE11) -> unconnected-(U3B-PT51B-PadE11)
- U3 pad E12: Net-(U3-PadE12) -> unconnected-(U3B-PT58B-PadE12)
- U3 pad E13: Net-(U3-PadE13) -> unconnected-(U3B-PT62B-PadE13)
- U3 pad E14: Net-(U3-PadE14) -> unconnected-(U3C-PR5C-PadE14)
- U3 pad E15: Net-(U3-PadE15) -> unconnected-(U3C-PR8B-PadE15)
- U3 pad E16: Net-(U3-PadE16) -> unconnected-(U3C-PR11D-PadE16)
- U3 pad E2: Net-(U3-PadE2) -> unconnected-(U3F-PL8B-PadE2)
- U3 pad E3: Net-(U3-PadE3) -> unconnected-(U3F-PL5C-PadE3)
- U3 pad E4: Net-(U3-PadE4) -> unconnected-(U3A-PT9A-PadE4)
- U3 pad E5: +3V3 -> unconnected-(U3A-PT13A-PadE5)
- U3 pad E6: Net-(U3-PadE6) -> unconnected-(U3A-PT20A-PadE6)
- U3 pad E7: Net-(U3-PadE7) -> unconnected-(U3A-GR00/PT24A-PadE7)
- U3 pad E8: Net-(U3-PadE8) -> unconnected-(U3B-PCK11/PT33A-PadE8)
- U3 pad E9: GND -> unconnected-(U3B-PT40B-PadE9)
- U3 pad F1: Net-(U3-PadF1) -> unconnected-(U3F-PL14A-PadF1)
- U3 pad F10: Net-(U3-PadF10) -> +3V3
- U3 pad F12: Net-(U3-PadF12) -> unconnected-(U3C-PR8D-PadF12)
- U3 pad F13: Net-(U3-PadF13) -> unconnected-(U3C-PR8C-PadF13)
- U3 pad F14: Net-(U3-PadF14) -> unconnected-(U3C-PR5D-PadF14)
- U3 pad F15: Net-(U3-PadF15) -> unconnected-(U3C-PR11C-PadF15)
- U3 pad F16: Net-(U3-PadF16) -> unconnected-(U3C-PR14A-PadF16)
- U3 pad F2: Net-(U3-PadF2) -> unconnected-(U3F-PL11C-PadF2)
- U3 pad F3: Net-(U3-PadF3) -> unconnected-(U3F-PL5D-PadF3)
- U3 pad F4: Net-(U3-PadF4) -> unconnected-(U3F-PL8C-PadF4)
- U3 pad F5: Net-(U3-PadF5) -> unconnected-(U3F-PL8D-PadF5)
- U3 pad F6: Net-(U3-PadF6) -> +3V3
- U3 pad F7: Net-(U3-PadF7) -> +3V3
- U3 pad F8: +3V3 -> GND
- U3 pad F9: Net-(U3-PadF9) -> GND
- U3 pad G1: Net-(U3-PadG1) -> unconnected-(U3F-GR71/PL20A-PadG1)
- U3 pad G10: +3V3 -> GND
- U3 pad G11: Net-(U3-PadG11) -> +2V5
- U3 pad G12: Net-(U3-PadG12) -> unconnected-(U3C-PR11A-PadG12)
- U3 pad G13: +3V3 -> unconnected-(U3C-PR11B-PadG13)
- U3 pad G14: Net-(U3-PadG14) -> unconnected-(U3C-Vref12/PR14C-PadG14)
- U3 pad G15: GND -> unconnected-(U3C-PR14B-PadG15)
- U3 pad G16: Net-(U3-PadG16) -> unconnected-(U3C-GR21/PR20A-PadG16)
- U3 pad G2: GND -> unconnected-(U3F-PL14B-PadG2)
- U3 pad G3: Net-(U3-PadG3) -> unconnected-(U3F-Vref17/PL14C-PadG3)
- U3 pad G4: +3V3 -> unconnected-(U3F-PL11B-PadG4)
- U3 pad G5: Net-(U3-PadG5) -> unconnected-(U3F-PL11A-PadG5)
- U3 pad G6: Net-(U3-PadG6) -> +1V1
- U3 pad G7: +1V2 -> +1V1
- U3 pad G9: +1V2 -> +1V1
- U3 pad H1: Net-(U3-PadH1) -> GND
- U3 pad H10: +1V2 -> GND
- U3 pad H11: Net-(U3-PadH11) -> +3V3
- U3 pad H12: GND -> unconnected-(U3C-PR17A-PadH12)
- U3 pad H13: Net-(U3-PadH13) -> unconnected-(U3C-PR17B-PadH13)
- U3 pad H14: Net-(U3-PadH14) -> unconnected-(U3C-PR14D-PadH14)
- U3 pad H15: Net-(U3-PadH15) -> unconnected-(U3C-PR20B-PadH15)
- U3 pad H16: Net-(U3-PadH16) -> GND
- U3 pad H2: Net-(U3-PadH2) -> unconnected-(U3F-PL20B-PadH2)
- U3 pad H3: Net-(U3-PadH3) -> unconnected-(U3F-PL14D-PadH3)
- U3 pad H4: Net-(U3-PadH4) -> unconnected-(U3F-PL17B-PadH4)
- U3 pad H5: Net-(U3-PadH5) -> unconnected-(U3F-PL17A-PadH5)
- U3 pad H7: GND -> +3V3
- U3 pad H8: +1V2 -> GND
- U3 pad J1: Net-(U3-PadJ1) -> unconnected-(U3F-PCK71/PL23A-PadJ1)
- U3 pad J10: +3V3 -> GND
- U3 pad J11: Net-(U3-PadJ11) -> +3V3
- U3 pad J12: Net-(U3-PadJ12) -> unconnected-(U3C-PR17D-PadJ12)
- U3 pad J13: Net-(U3-PadJ13) -> unconnected-(U3C-PR17C-PadJ13)
- U3 pad J14: Net-(U3-PadJ14) -> unconnected-(U3C-GR20/PR20C-PadJ14)
- U3 pad J15: +3V3 -> unconnected-(U3C-~{PCK}21/PR23B-PadJ15)
- U3 pad J16: Net-(U3-PadJ16) -> unconnected-(U3C-PCK21/PR23A-PadJ16)
- U3 pad J2: +3V3 -> unconnected-(U3F-~{PCK}71/PL23B-PadJ2)
- U3 pad J3: Net-(U3-PadJ3) -> unconnected-(U3F-GR70/PL20C-PadJ3)
- U3 pad J4: Net-(U3-PadJ4) -> unconnected-(U3F-PL17C-PadJ4)
- U3 pad J5: GND -> unconnected-(U3F-PL17D-PadJ5)
- U3 pad J6: Net-(U3-PadJ6) -> +3V3
- U3 pad J7: +1V2 -> +3V3
- U3 pad J9: +1V2 -> GND
- U3 pad K1: Net-(U3-PadK1) -> unconnected-(U3F-PCK70/PL23C-PadK1)
- U3 pad K10: +1V2 -> GND
- U3 pad K11: Net-(U3-PadK11) -> +3V3
- U3 pad K12: Net-(U3-PadK12) -> unconnected-(U3D-PR29B-PadK12)
- U3 pad K13: +3V3 -> unconnected-(U3D-GR30/PR29A-PadK13)
- U3 pad K14: Net-(U3-PadK14) -> unconnected-(U3C-PR20D-PadK14)
- U3 pad K15: Net-(U3-PadK15) -> unconnected-(U3C-~{PCK}20/PR23D-PadK15)
- U3 pad K16: Net-(U3-PadK16) -> unconnected-(U3C-PCK20/PR23C-PadK16)
- U3 pad K2: Net-(U3-PadK2) -> unconnected-(U3F-~{PCK}70/PL23D-PadK2)
- U3 pad K3: Net-(U3-PadK3) -> unconnected-(U3F-PL20D-PadK3)
- U3 pad K4: +3V3 -> unconnected-(U3E-GR60/PL29A-PadK4)
- U3 pad K5: Net-(U3-PadK5) -> unconnected-(U3E-PL29B-PadK5)
- U3 pad K6: Net-(U3-PadK6) -> GND
- U3 pad K8: +1V2 -> GND
- U3 pad L1: Net-(U3-PadL1) -> unconnected-(U3E-PCK61/PL26A-PadL1)
- U3 pad L10: Net-(U3-PadL10) -> +1V1
- U3 pad L11: Net-(U3-PadL11) -> +3V3
- U3 pad L12: Net-(U3-PadL12) -> unconnected-(U3D-PR29D-PadL12)
- U3 pad L13: Net-(U3-PadL13) -> unconnected-(U3D-GR31/PR26C-PadL13)
- U3 pad L14: Net-(U3-PadL14) -> unconnected-(U3D-PR32C-PadL14)
- U3 pad L15: GND -> unconnected-(U3D-~{PCK}31/PR26B-PadL15)
- U3 pad L16: Net-(U3-PadL16) -> unconnected-(U3D-PCK31/PR26A-PadL16)
- U3 pad L2: GND -> unconnected-(U3E-~{PCK}61/PL26B-PadL2)
- U3 pad L3: Net-(U3-PadL3) -> unconnected-(U3E-PL32C-PadL3)
- U3 pad L4: Net-(U3-PadL4) -> unconnected-(U3E-GR61/PL29C-PadL4)
- U3 pad L5: Net-(U3-PadL5) -> unconnected-(U3E-PL29D-PadL5)
- U3 pad L7: Net-(U3-PadL7) -> +2V5
- U3 pad L8: Net-(U3-PadL8) -> +1V1
- U3 pad L9: +3V3 -> +1V1
- U3 pad M1: Net-(U3-PadM1) -> unconnected-(U3E-PCK60/PL26C-PadM1)
- U3 pad M11: Net-(U3-PadM11) -> unconnected-(U3D-PR47A-PadM11)
- U3 pad M12: Net-(U3-PadM12) -> unconnected-(U3D-PR44C-PadM12)
- U3 pad M13: Net-(U3-PadM13) -> unconnected-(U3D-PR35C-PadM13)
- U3 pad M14: Net-(U3-PadM14) -> unconnected-(U3D-PR32D-PadM14)
- U3 pad M15: Net-(U3-PadM15) -> unconnected-(U3D-~{PCK}30/PR26D-PadM15)
- U3 pad M16: Net-(U3-PadM16) -> unconnected-(U3D-PCK30/PR26C-PadM16)
- U3 pad M2: Net-(U3-PadM2) -> unconnected-(U3E-~{PCK}60/PL26D-PadM2)
- U3 pad M3: Net-(U3-PadM3) -> unconnected-(U3E-PL32D-PadM3)
- U3 pad M4: Net-(U3-PadM4) -> unconnected-(U3E-PL35C-PadM4)
- U3 pad M5: Net-(U3-PadM5) -> unconnected-(U3E-PL44C-PadM5)
- U3 pad M6: Net-(U3-PadM6) -> unconnected-(U3E-PL47A-PadM6)
- U3 pad M7: Net-(U3-PadM7) -> unconnected-(U3G-PB9B/D2-PadM7)
- U3 pad M8: GND -> /Control/~{CSO}
- U3 pad M9: Net-(U3-PadM9) -> unconnected-(U3G-~{WRITE}/PB18A-PadM9)
- U3 pad N1: Net-(U3-PadN1) -> unconnected-(U3E-PL32A-PadN1)
- U3 pad N10: +3V3 -> unconnected-(U3G-CFG0-PadN10)
- U3 pad N11: /Control/M1 -> unconnected-(U3D-PR47B-PadN11)
- U3 pad N12: Net-(U3-PadN12) -> unconnected-(U3D-PR44D-PadN12)
- U3 pad N13: GND -> unconnected-(U3D-PR38A-PadN13)
- U3 pad N14: Net-(U3-PadN14) -> unconnected-(U3D-PR35D-PadN14)
- U3 pad N15: +3V3 -> GND
- U3 pad N16: Net-(U3-PadN16) -> unconnected-(U3D-PR32A-PadN16)
- U3 pad N2: +3V3 -> GND
- U3 pad N3: Net-(U3-PadN3) -> unconnected-(U3E-PL35D-PadN3)
- U3 pad N4: Net-(U3-PadN4) -> unconnected-(U3E-PL38A-PadN4)
- U3 pad N5: Net-(U3-PadN5) -> unconnected-(U3E-PL44D-PadN5)
- U3 pad N6: Net-(U3-PadN6) -> unconnected-(U3E-PL47B-PadN6)
- U3 pad N7: +3V3 -> unconnected-(U3G-PB9A/D3-PadN7)
- U3 pad N8: Net-(U3-PadN8) -> unconnected-(U3G-M~{CS}/PB15A-PadN8)
- U3 pad N9: Net-(U3-PadN9) -> /Control/CCLK
- U3 pad P1: Net-(U3-PadP1) -> unconnected-(U3E-PL35A-PadP1)
- U3 pad P10: /Control/MOSI_DIN -> unconnected-(U3G-CFG1-PadP10)
- U3 pad P11: Net-(U3-PadP11) -> unconnected-(U3D-RPLL0/PR47C-PadP11)
- U3 pad P12: Net-(U3-PadP12) -> unconnected-(U3D-~{RPLL}0/PR47D-PadP12)
- U3 pad P13: /Control/DONE -> unconnected-(U3D-PR41A-PadP13)
- U3 pad P14: Net-(U3-PadP14) -> unconnected-(U3D-PR38B-PadP14)
- U3 pad P15: Net-(U3-PadP15) -> unconnected-(U3D-PR32B-PadP15)
- U3 pad P16: Net-(U3-PadP16) -> unconnected-(U3D-PR35A-PadP16)
- U3 pad P2: Net-(U3-PadP2) -> unconnected-(U3E-PL32B-PadP2)
- U3 pad P3: GND -> unconnected-(U3E-PL38B-PadP3)
- U3 pad P4: Net-(U3-PadP4) -> unconnected-(U3E-PL41A-PadP4)
- U3 pad P5: Net-(U3-PadP5) -> unconnected-(U3E-~{RPLL}0/PL47D-PadP5)
- U3 pad P6: Net-(U3-PadP6) -> unconnected-(U3E-RPLL0/PL47C-PadP6)
- U3 pad P7: Net-(U3-PadP7) -> unconnected-(U3G-MOSI2/PB6B-PadP7)
- U3 pad P8: Net-(U3-PadP8) -> unconnected-(U3G-S~{CS}1/PB13B-PadP8)
- U3 pad P9: Net-(U3-PadP9) -> /Control/DONE
- U3 pad R1: Net-(U3-PadR1) -> unconnected-(U3E-Vref16/PL35B-PadR1)
- U3 pad R10: GND -> unconnected-(U3G-CFG2-PadR10)
- U3 pad R12: Net-(U3-PadR12) -> unconnected-(U3D-PR44A-PadR12)
- U3 pad R13: +3V3 -> unconnected-(U3D-PR41C-PadR13)
- U3 pad R14: Net-(U3-PadR14) -> unconnected-(U3D-PR41B-PadR14)
- U3 pad R15: Net-(U3-PadR15) -> unconnected-(U3D-PR38C-PadR15)
- U3 pad R16: Net-(U3-PadR16) -> unconnected-(U3D-Vref13/PR35B-PadR16)
- U3 pad R2: Net-(U3-PadR2) -> unconnected-(U3E-PL38C-PadR2)
- U3 pad R3: /Control/~INIT~ -> unconnected-(U3E-PL41B-PadR3)
- U3 pad R4: +3V3 -> unconnected-(U3E-PL41C-PadR4)
- U3 pad R5: Net-(U3-PadR5) -> unconnected-(U3E-PL44A-PadR5)
- U3 pad R6: GND -> unconnected-(U3G-PB4B-PadR6)
- U3 pad R7: Net-(U3-PadR7) -> unconnected-(U3G-MISO2/PB6A-PadR7)
- U3 pad R8: +3V3 -> unconnected-(U3G-S~{CS}/PB13A-PadR8)
- U3 pad T12: Net-(U3-PadT12) -> GND
- U3 pad T13: Net-(U3-PadT13) -> unconnected-(U3D-PR44B-PadT13)
- U3 pad T14: Net-(U3-PadT14) -> unconnected-(U3D-PR41D-PadT14)
- U3 pad T15: Net-(U3-PadT15) -> unconnected-(U3D-PR38D-PadT15)
- U3 pad T2: /Control/~PROG~ -> unconnected-(U3E-PL38D-PadT2)
- U3 pad T3: Net-(U3-PadT3) -> unconnected-(U3E-PL41D-PadT3)
- U3 pad T4: Net-(U3-PadT4) -> unconnected-(U3E-PL44B-PadT4)
- U3 pad T5: Net-(U3-PadT5) -> GND
- U3 pad T6: Net-(U3-PadT6) -> unconnected-(U3G-PB4A-PadT6)
- U5 pad 16: /Control/RAM_~WE~ -> /Control/RAM_~{WE}
- U5 pad 17: /Control/RAM_~CAS~ -> /Control/RAM_~{CAS}
- U5 pad 18: /Control/RAM_~RAS~ -> /Control/RAM_~{RAS}
- U5 pad 19: /Control/RAM_~CS~ -> /Control/RAM_~{CS}
- U6 pad 1: GND -> /Control/IOA~{OE}
- U6 pad 11: GND -> +5V
- U6 pad 12: /PDSBuf/FSB_~RESET~ -> unconnected-(U6-Q7-Pad12)
- U6 pad 13: GND -> unconnected-(U6-Q6-Pad13)
- U6 pad 14: /Control/IOB_~BERR~ -> unconnected-(U6-Q5-Pad14)
- U6 pad 15: /PDS/C16M -> unconnected-(U6-Q4-Pad15)
- U6 pad 16: /Control/IOB_~HALT~ -> /PDS/A1
- U6 pad 17: /PDSBuf/IOB_~DSACK~1 -> /PDS/A0
- U6 pad 18: /Control/IOB_~DSACK~0 -> /PDS/~{RMC}
- U6 pad 19: GND -> /PDS/FC0
- U6 pad 2: /PDSBuf/IOB_~RESET~ -> /PDSBuf/LFC0
- U6 pad 20: +3V3 -> +5V
- U6 pad 4: /PDSBuf/IOB_~BERR~ -> unconnected-(U6-D2-Pad4)
- U6 pad 5: /Control/IOB_C16M -> unconnected-(U6-D3-Pad5)
- U6 pad 6: /PDSBuf/IOB_~HALT~ -> unconnected-(U6-D4-Pad6)
- U6 pad 7: Net-(U13-Pad7) -> unconnected-(U6-D5-Pad7)
- U6 pad 8: /PDSBuf/IOB_~DSACK~0 -> unconnected-(U6-D6-Pad8)
- U6 pad 9: Net-(U13-Pad9) -> unconnected-(U6-D7-Pad9)
- U8 pad 1: /PDSBuf/A~OE~ -> GND
- U8 pad 11: +5V -> /PDSBuf/SoutLE
- U8 pad 12: /PDSBuf/IOB_~DS~ -> unconnected-(U8-Q7-Pad12)
- U8 pad 14: /PDS/A0 -> /PDS/~{BR}
- U8 pad 15: /PDS/A1 -> /PDSBuf/L~{IRQ}
- U8 pad 16: /PDS/A2 -> /PDSBuf/LFC0
- U8 pad 17: /PDS/A3 -> /PDSBuf/LFC1
- U8 pad 18: /PDSBuf/IOB_SIZ0 -> /PDSBuf/LFC2
- U8 pad 2: /PDSBuf/IOC_SIZ1 -> /PDSBuf/AD7
- U8 pad 3: /PDSBuf/IOC_SIZ0 -> /PDSBuf/AD6
- U8 pad 4: /PDSBuf/IOC_A3 -> /PDSBuf/AD5
- U8 pad 5: /PDSBuf/IOC_A2 -> /PDSBuf/AD4
- U8 pad 6: /PDSBuf/IOC_A1 -> /PDSBuf/AD3
- U8 pad 8: /Control/IOC_~AS~ -> /PDSBuf/AD1
- U8 pad 9: /Control/IOC_~DS~ -> /PDSBuf/AD0
- U9 pad 1: /PDSBuf/A~OE~ -> /Control/IOA~{OE}
- U9 pad 11: /PDSBuf/ADoutLE -> /PDSBuf/AoutLE
- U9 pad 12: /PDS/A24 -> /PDS/A13
- U9 pad 13: /PDS/A25 -> /PDS/A11
- U9 pad 14: /PDS/A26 -> /PDS/A5
- U9 pad 15: /PDS/A27 -> /PDS/A12
- U9 pad 16: /PDS/A30 -> /PDS/A6
- U9 pad 17: /PDS/A31 -> /PDS/A3
- U9 pad 18: /PDSBuf/IOB_R~W~ -> /PDS/A2
- U9 pad 19: Net-(U9-Pad19) -> /PDS/A4
- U9 pad 2: GND -> /PDSBuf/FSB_A27
- U9 pad 3: /CPUBuf/FSB_R~W~ -> /PDSBuf/FSB_A27
- U9 pad 4: /CPUBuf/FSB_A31 -> /PDSBuf/FSB_A26
- U9 pad 5: /CPUBuf/FSB_A30 -> /PDSBuf/FSB_A25
- U9 pad 6: /CPUBuf/FSB_A27 -> /PDSBuf/FSB_A27
- U9 pad 7: /CPUBuf/FSB_A26 -> /PDSBuf/FSB_A26
- U9 pad 8: /CPUBuf/FSB_A25 -> /PDSBuf/FSB_A25
- U9 pad 9: /CPUBuf/FSB_A24 -> /PDSBuf/FSB_A24
Routing:
- net (no net): track 1050.8 -> 31.0 mm, vias 160 -> 16
- net +1V2: track 226.4 -> 0.00 mm, vias 24 -> 0
- net /Control/CPUCLK: track 129.2 -> 0.00 mm
- net /Control/FPUCLK: track 82.9 -> 0.00 mm
- net /CPUBuf/CPU_~DS~: track 66.3 -> 0.00 mm, vias 1 -> 0
- net /CPUBuf/CPU_~AS~: track 64.8 -> 0.00 mm, vias 1 -> 0
- net +3V3: track 34.2 -> 98.7 mm, vias 36 -> 89
- net /CPUBuf/CPU_~DSACK~0: track 63.5 -> 0.00 mm, vias 1 -> 0
- net /CPUBuf/CPU_~DSACK~1: track 63.3 -> 0.00 mm, vias 1 -> 0
- net +5V: track 170.5 -> 109.1 mm, vias 136 -> 73
- net /CPUBuf/CPU_R~W~: track 56.1 -> 0.00 mm, vias 1 -> 0
- net /CPUBuf/CPU_D8: track 73.7 -> 20.7 mm, vias 2 -> 1
- net /CPUBuf/CPU_D9: track 76.5 -> 24.3 mm, vias 2 -> 1
- net /CPUBuf/CPU_D13: track 70.5 -> 18.6 mm, vias 2 -> 1
- net /CPUBuf/CPU_D15: track 70.6 -> 19.2 mm, vias 2 -> 1
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- added copper zone on In3.Cu, net +1V1
- added copper zone on In2.Cu, net +5V
- added copper zone on In3.Cu, net GND
- added copper zone on In4.Cu, net GND
- removed copper zone on F.Cu, net GND
Other:
- board size 82.7 x 136.5 mm -> 108.1 x 136.5 mm
- copper layers 4 -> 6
- net class Default removed

Commit message: idk
Parts:
- removed the REF** at (167.1, 70.8)
- removed the REF** at (182.3, 64.8)
- removed the REF** at (167.1, 60.8)
- removed the REF** at (182.3, 69.5)
- removed the REF** at (167.1, 63.4)
- removed the REF** at (192.9, 70.9)
- removed the REF** at (167.1, 67.2)
- removed the REF** at (167.1, 81.5)
- removed the U4 at (174.7, 71.7)
Routing:
- net +5V: track 109.1 -> 82.1 mm, vias 73 -> 51
- net GND: track 216.6 -> 189.8 mm, vias 254 -> 229
- net /RAM/RA4: track 7.51 -> 1.70 mm
- net /RAM/D5: track 3.84 -> 1.90 mm
- net /RAM/D4: track 3.04 -> 1.10 mm
- net /RAM/D1: track 3.04 -> 1.10 mm
- net /RAM/D6: track 3.84 -> 1.90 mm
- net /RAM/D3: track 3.04 -> 1.10 mm
- net /RAM/D2: track 3.04 -> 1.10 mm
- net /RAM/D11: track 3.84 -> 1.90 mm
- net /RAM/D10: track 3.04 -> 1.10 mm
- net /RAM/D14: track 3.04 -> 1.10 mm
- net /RAM/D13: track 3.84 -> 1.90 mm
- net /RAM/D9: track 3.04 -> 1.10 mm
- net /RAM/D12: track 3.04 -> 1.10 mm
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