File: SE-030.kicad_sch (KiCad schematic)
At the start: 10 parts, among them J1 Micro_SD_Card_Det1

Commit message: idk
Other:
- removed sheet VDAC
- removed sheet VidControl
- note added: "SE/30: RAMCLK[5:2] RAM~{CS}[2:1] SD[3:0] SDPWR"
- note removed: "SE/30: RAMCLK[5:2] RAM~{CS}[2:1] SD[3:0] SDPWR VD[6:0] VCLK"
Changed lines of the file:
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@@
     (stroke (width 0) (type default))
   )
-  (text "SE/30:\n\nRAMCLK[5:2]\nRAM~{CS}[2:1]\n\nSD[3:0]\nSDPWR\n\nVD[6:0]\nVCLK\n"
-    (at 38.1 71.12 0)
+  (text "SE/30:\n\nRAMCLK[5:2]\nRAM~{CS}[2:1]\n\nSD[3:0]\nSDPWR" (at 38.1 71.12 0)
     (effects (font (size 1.27 1.27)) (justify left bottom))
   )
@@
       )
     )
-  )
-  (sheet (at 104.14 68.58) (size 22.86 15.24) (fields_autoplaced)
-    (stroke (width 0.1524) (type solid))
-    (fill (color 0 0 0 0.0000))
-    (property "Sheetname" "VidControl" (at 104.14 67.8684 0)
-      (effects (font (size 1.27 1.27)) (justify left bottom))
-    )
-    (property "Sheetfile" "VidControl.kicad_sch" (at 104.14 84.4046 0)
-      (effects (font (size 1.27 1.27)) (justify left top))
-    )
-    (pin "VD[6..0]" input (at 104.14 76.2 180)
-      (effects (font (size 1.27 1.27)) (justify left))
-    )
-    (pin "VCLK" input (at 104.14 71.12 180)
-      (effects (font (size 1.27 1.27)) (justify left))
-    )
-    (pin "G[5..0]" output (at 127 73.66 0)
-      (effects (font (size 1.27 1.27)) (justify right))
-    )
-    (pin "R[5..0]" output (at 127 71.12 0)
-      (effects (font (size 1.27 1.27)) (justify right))
-    )
-    (pin "B[5..0]" output (at 127 76.2 0)
-      (effects (font (size 1.27 1.27)) (justify right))
-    )
-    (pin "~{VSYNC}" output (at 127 81.28 0)
-      (effects (font (size 1.27 1.27)) (justify right))
-    )
-    (pin "~{HSYNC}" output (at 127 78.74 0)
-      (effects (font (size 1.27 1.27)) (justify right))
-    )
-    (instances
-      (project "SE-030"
-        (path "/70f3c4d7-2986-471b-b5fa-d888368dbdd8" (page "8"))
-      )
-    )
-  )
-  (sheet (at 129.54 68.58) (size 17.78 15.24) (fields_autoplaced)
-    (stroke (width 0.1524) (type solid))
-    (fill (color 0 0 0 0.0000))
-    (property "Sheetname" "VDAC" (at 129.54 67.8684 0)
-      (effects (font (size 1.27 1.27)) (justify left bottom))
-    )
-    (property "Sheetfile" "VDAC.kicad_sch" (at 129.54 84.4046 0)
-      (effects (font (size 1.27 1.27)) (justify left top))
-    )
-    (pin "~{VSYNC}o" output (at 147.32 81.28 0)
-      (effects (font (size 1.27 1.27)) (justify right))
-    )
-    (pin "Ro" output (at 147.32 71.12 0)
-      (effects (font (size 1.27 1.27)) (justify right))
-    )
-    (pin "Go" output (at 147.32 73.66 0)
-      (effects (font (size 1.27 1.27)) (justify right))
-    )
-    (pin "~{HSYNC}o" output (at 147.32 78.74 0)
-      (effects (font (size 1.27 1.27)) (justify right))
-    )
-    (pin "Bo" output (at 147.32 76.2 0)
-      (effects (font (size 1.27 1.27)) (justify right))
-    )
-    (pin "~{HSYNC}i" input (at 129.54 78.74 180)
-      (effects (font (size 1.27 1.27)) (justify left))
-    )
-    (pin "Gi[5..0]" input (at 129.54 73.66 180)
-      (effects (font (size 1.27 1.27)) (justify left))
-    )
-    (pin "Bi[5..0]" input (at 129.54 76.2 180)
-      (effects (font (size 1.27 1.27)) (justify left))
-    )
-    (pin "~{VSYNC}i" input (at 129.54 81.28 180)
-      (effects (font (size 1.27 1.27)) (justify left))
-    )
-    (pin "Ri[5..0]" input (at 129.54 71.12 180)
-      (effects (font (size 1.27 1.27)) (justify left))
-    )
-    (instances
-      (project "SE-030"
-        (path "/70f3c4d7-2986-471b-b5fa-d888368dbdd8" (page "9"))
-      )
-    )
